Commit message: Completion of ddrive robot for rviz use

File: diff_drive/urdf/ddrive.urdf.xacro (robot description, xacro)
@@ -1,24 +1,17 @@
 <?xml version="1.0"?>
 <robot xmlns:xacro="http://wiki.ros.org/wiki/xacro" name="ddrive">
-<!-- <xacro:property name="arm" value="$(find homework2)/config/arm.yaml" />
-<xacro:property name="dictionary" value="${load_yaml(arm)}" />
-<xacro:property name="L1" value="${dictionary['L1']}" />
-<xacro:property name="L2" value="${dictionary['L2']}" />
-<xacro:property name="R1" value="${dictionary['R1']}" />
-<xacro:property name="R2" value="${dictionary['R2']}" />
-<xacro:property name="m" value="1" /> -->
-<link name="base_link" >
-    <visual>
-    <origin xyz="0 0 0" rpy="0 0 0" />
-        <geometry>
-            <cylinder radius="0.1" length="0.1"/>
-        </geometry>
-        <material name="transparent_mat">
-            <color rgba="1 1 1 0" />
-        </material>
-    </visual>
-</link>
+<xacro:property name="ddrive" value="$(find diff_drive)/config/ddrive.yaml" />
+<xacro:property name="config" value="${load_yaml(ddrive)}" />
+<xacro:property name="box_l" value="${config['box_l']}" />
+<xacro:property name="box_w" value="${config['box_w']}" />
+<xacro:property name="box_h" value="${config['box_h']}" />
+<xacro:property name="box_m" value="${config['box_m']}" />
+<xacro:property name="wheel_h" value="${config['wheel_h']}" />
+<xacro:property name="wheel_r" value="${config['wheel_r']}" />
+<xacro:property name="wheel_m" value="${config['wheel_m']}" />
+<xacro:property name="caster_r" value="${config['caster_r']}" />
+<xacro:property name="caster_m" value="${config['caster_m']}" />
+<link name="base_link" />
 <joint name ="base" type="fixed">
-    <axis xyz="0 0 0" />
     <origin xyz="0 0 0" rpy="0 0 0" />
     <parent link="base_link" />
@@ -29,5 +22,5 @@
         <origin rpy="0 0 0" xyz="0 0 0" />
         <geometry>
-            <box size="0.5 0.3 0.1" />
+            <box size="${box_l} ${box_w} ${box_h}" />
         </geometry>
         <material name="black">
@@ -35,18 +28,18 @@
         </material>
         <inertial>
-            <mass value="5.0" />
+            <mass value="${box_m}" />
             <origin rpy="0 0 0" xyz="0 0 0.1" />
-            <inertia ixx="1/12*${5.0}*(${0.1}**2 + ${0.5}**2)" ixy="0.0" ixz="0.0" iyy="1/12*${5.0}*(${0.3}**2 + ${0.5}**2)" iyz="0.0" izz="1/12*${5.0}*(${0.3}**2 + ${0.1}**2)"/>
+            <inertia ixx="1/12*${box_m}*(${box_h}**2 + ${box_l}**2)" ixy="0.0" ixz="0.0" iyy="1/12*${box_m}*(${box_w}**2 + ${box_l}**2)" iyz="0.0" izz="1/12*${box_m}*(${box_w}**2 + ${box_h}**2)"/>
         </inertial>
     </visual>
     <collision>
         <geometry>
-            <box size="0.5 0.3 0.1"/>
+            <box size="${box_l} ${box_w} ${box_h}"/>
         </geometry>
     </collision>
 </link>
-<joint name="right" type="continuous">
+<joint name="wheel_right" type="continuous">
     <axis xyz="0 1 0" />
-    <origin xyz="0.1875 -0.15 0" rpy="0 0 0" />
+    <origin xyz="0.1875 -0.17 0" rpy="0 0 0" />
     <parent link="chassis" />
     <child link="right_wheel" />
@@ -56,23 +49,23 @@
     <origin rpy="0 ${pi/2} ${pi/2}" xyz="0 0 0" />
         <geometry>
-            <cylinder length="0.04" radius="0.15"/>
+            <cylinder length="${wheel_h}" radius="${wheel_r}"/>
         </geometry>
-        <material name="green_mat">
-            <color rgba="0 1 0 1" />
+        <material name="gray">
+            <color rgba="0.3 0.3 0.3 1.0" />
         </material>
         <inertial>
-           <mass value="0.2"/>
-           <inertia ixx="1/12*${0.2}*(3*${0.15}**2 + ${0.04}**2)" ixy="0.0" ixz="0.0" iyy="1/12*${0.2}*(3*${0.15}**2 + ${0.04}**2)" iyz="0.0" izz="1/2*${0.2}*${0.15}**2"/>
+           <mass value="${wheel_m}"/>
+           <inertia ixx="1/12*${wheel_m}*(3*${wheel_r}**2 + ${wheel_h}**2)" ixy="0.0" ixz="0.0" iyy="1/12*${wheel_m}*(3*${wheel_r}**2 + ${wheel_h}**2)" iyz="0.0" izz="1/2*${wheel_m}*${wheel_r}**2"/>
          </inertial>
     </visual>
     <collision>
            <geometry>
-             <cylinder length="0.04" radius="0.15"/>
+             <cylinder length="${wheel_h}" radius="${wheel_r}"/>
            </geometry>
     </collision>
 </link>
-<joint name="left" type="continuous">
+<joint name="wheel_left" type="continuous">
     <axis xyz="0 1 0" />
-    <origin xyz="0.1875 0.15 0" rpy="0 0 0" />
+    <origin xyz="0.1875 0.17 0" rpy="0 0 0" />
     <parent link="chassis" />
     <child link="left_wheel" />
@@ -82,17 +75,67 @@
     <origin rpy="0 ${pi/2} ${pi/2}" xyz="0 0 0" />
         <geometry>
-            <cylinder length="0.04" radius="0.15"/>
+            <cylinder length="${wheel_h}" radius="${wheel_r}"/>
         </geometry>
-        <material name="green_mat">
-            <color rgba="0 1 0 1" />
+        <material name="gray">
+            <color rgba="0.3 0.3 0.3 1.0" />
         </material>
         <inertial>
            <mass value="0.2"/>
-           <inertia ixx="1/12*${0.2}*(3*${0.15}**2 + ${0.04}**2)" ixy="0.0" ixz="0.0" iyy="1/12*${0.2}*(3*${0.15}**2 + ${0.04}**2)" iyz="0.0" izz="1/2*${0.2}*${0.15}**2"/>
+           <inertia ixx="1/12*${wheel_m}*(3*${wheel_r}**2 + ${wheel_h}**2)" ixy="0.0" ixz="0.0" iyy="1/12*${wheel_m}*(3*${wheel_r}**2 + ${wheel_h}**2)" iyz="0.0" izz="1/2*${wheel_m}*${wheel_r}**2"/>
          </inertial>
     </visual>
     <collision>
            <geometry>
-             <cylinder length="0.04" radius="0.15"/>
+             <cylinder length="${wheel_h}" radius="${wheel_r}"/>
+           </geometry>
+    </collision>
+</link>
+<joint name="caster_top" type="fixed">
+    <origin xyz="-0.1875 0 0.1" rpy="0 0 0" />
+    <parent link="chassis" />
+    <child link="caster_top" />
+</joint>
+<link name="caster_top">
+    <visual>
+    <origin rpy="${pi/2} 0 0" xyz="0 0 0" />
+        <geometry>
+            <sphere radius="${caster_r}"/>
+        </geometry>
+        <material name="gray">
+            <color rgba="0.3 0.3 0.3 1" />
+        </material>
+        <inertial>
+           <mass value="${caster_m}"/>
+           <inertia ixx="2/5*${caster_m}*(${caster_r}**2)" ixy="0.0" ixz="0.0" iyy="2/5*${caster_m}*(${caster_r}**2)" iyz="0.0" izz="2/5*${caster_m}*${caster_r}**2"/>
+         </inertial>
+    </visual>
+    <collision>
+           <geometry>
+             <sphere radius="${caster_r}"/>
+           </geometry>
+    </collision>
+</link>
+<joint name="caster_bottom" type="fixed">
+    <origin xyz="-0.1875 0 -0.1" rpy="0 0 0" />
+    <parent link="chassis" />
+    <child link="caster_bottom" />
+</joint>
+<link name="caster_bottom">
+    <visual>
+    <origin rpy="${pi/2} 0 0" xyz="0 0 0" />
+        <geometry>
+            <sphere radius="${caster_r}"/>
+        </geometry>
+        <material name="gray">
+            <color rgba="0.3 0.3 0.3 1" />
+        </material>
+        <inertial>
+           <mass value="0.05"/>
+           <inertia ixx="2/5*${caster_m}*(${caster_r}**2)" ixy="0.0" ixz="0.0" iyy="2/5*${caster_m}*(${caster_r}**2)" iyz="0.0" izz="2/5*${caster_m}*${caster_r}**2"/>
+         </inertial>
+    </visual>
+    <collision>
+           <geometry>
+             <sphere radius="${caster_r}"/>
            </geometry>
     </collision>

Commit message: Initial creation of gazebo urdf to hold gazebo properties.

File: diff_drive/urdf/ddrive.urdf.xacro (robot description, xacro)
@@ -12,4 +12,10 @@
 <xacro:property name="caster_r" value="${config['caster_r']}" />
 <xacro:property name="caster_m" value="${config['caster_m']}" />
+<material name="black">
+    <color rgba="0 0 0 1"/>
+</material>
+<material name="gray">
+    <color rgba="0.3 0.3 0.3 1" />
+</material>
 <link name="base_link" />
 <joint name ="base" type="fixed">
@@ -24,7 +30,5 @@
             <box size="${box_l} ${box_w} ${box_h}" />
         </geometry>
-        <material name="black">
-            <color rgba="0 0 0 1"/>
-        </material>
+        <material name="black"/>
         <inertial>
             <mass value="${box_m}" />
@@ -51,7 +55,5 @@
             <cylinder length="${wheel_h}" radius="${wheel_r}"/>
         </geometry>
-        <material name="gray">
-            <color rgba="0.3 0.3 0.3 1.0" />
-        </material>
+        <material name="gray"/>
         <inertial>
            <mass value="${wheel_m}"/>
@@ -77,7 +79,5 @@
             <cylinder length="${wheel_h}" radius="${wheel_r}"/>
         </geometry>
-        <material name="gray">
-            <color rgba="0.3 0.3 0.3 1.0" />
-        </material>
+        <material name="gray"/>
         <inertial>
            <mass value="0.2"/>
@@ -102,7 +102,5 @@
             <sphere radius="${caster_r}"/>
         </geometry>
-        <material name="gray">
-            <color rgba="0.3 0.3 0.3 1" />
-        </material>
+        <material name="gray"/>
         <inertial>
            <mass value="${caster_m}"/>
@@ -127,7 +125,5 @@
             <sphere radius="${caster_r}"/>
         </geometry>
-        <material name="gray">
-            <color rgba="0.3 0.3 0.3 1" />
-        </material>
+        <material name="gray"/>
         <inertial>
            <mass value="0.05"/>

Commit message: Updated inertial tags in ddrive urdf, need to correct the rest

File: diff_drive/urdf/ddrive.urdf.xacro (robot description, xacro)
@@ -32,15 +32,18 @@
         </geometry>
         <material name="black"/>
-        <inertial>
-            <mass value="${box_m}" />
-            <origin rpy="0 0 0" xyz="0 0 0.1" />
-            <inertia ixx="1/12*${box_m}*(${box_h}**2 + ${box_l}**2)" ixy="0.0" ixz="0.0" iyy="1/12*${box_m}*(${box_w}**2 + ${box_l}**2)" iyz="0.0" izz="1/12*${box_m}*(${box_w}**2 + ${box_h}**2)"/>
-        </inertial>
     </visual>
     <collision>
+        <origin rpy="0 0 0" xyz="0 0 0" />
         <geometry>
             <box size="${box_l} ${box_w} ${box_h}"/>
         </geometry>
     </collision>
+    <inertial>
+        <origin rpy="0 0 0" xyz="0 0 0" />
+        <mass value="${box_m}" />
+        <inertia ixx="${1/12*box_m*(box_h**2 + box_l**2)}" ixy="0.0" ixz="0.0"
+                 iyy="${1/12*box_m*(box_h**2 + box_l**2)}" iyz="0.0"
+                 izz="${1/12*box_m*(box_w**2 + box_h**2)}"/>
+    </inertial>
 </link>
 <joint name="wheel_right" type="continuous">
@@ -59,11 +62,13 @@
         <inertial>
            <mass value="${wheel_m}"/>
+           <origin rpy="0 0 0" xyz="0 0 0" />
            <inertia ixx="1/12*${wheel_m}*(3*${wheel_r}**2 + ${wheel_h}**2)" ixy="0.0" ixz="0.0" iyy="1/12*${wheel_m}*(3*${wheel_r}**2 + ${wheel_h}**2)" iyz="0.0" izz="1/2*${wheel_m}*${wheel_r}**2"/>
          </inertial>
     </visual>
     <collision>
-           <geometry>
-             <cylinder length="${wheel_h}" radius="${wheel_r}"/>
-           </geometry>
+        <origin rpy="0 0 0" xyz="0 0 0" />
+        <geometry>
+            <cylinder length="${wheel_h}" radius="${wheel_r}"/>
+        </geometry>
     </collision>
 </link>
@@ -83,11 +88,13 @@
         <inertial>
            <mass value="0.2"/>
+           <origin rpy="0 0 0" xyz="0 0 0" />
            <inertia ixx="1/12*${wheel_m}*(3*${wheel_r}**2 + ${wheel_h}**2)" ixy="0.0" ixz="0.0" iyy="1/12*${wheel_m}*(3*${wheel_r}**2 + ${wheel_h}**2)" iyz="0.0" izz="1/2*${wheel_m}*${wheel_r}**2"/>
          </inertial>
     </visual>
     <collision>
-           <geometry>
-             <cylinder length="${wheel_h}" radius="${wheel_r}"/>
-           </geometry>
+        <origin rpy="0 0 0" xyz="0 0 0" />
+        <geometry>
+            <cylinder length="${wheel_h}" radius="${wheel_r}"/>
+        </geometry>
     </collision>
 </link>
@@ -106,11 +113,13 @@
         <inertial>
            <mass value="${caster_m}"/>
+           <origin xyz="0 0 0" />
            <inertia ixx="2/5*${caster_m}*(${caster_r}**2)" ixy="0.0" ixz="0.0" iyy="2/5*${caster_m}*(${caster_r}**2)" iyz="0.0" izz="2/5*${caster_m}*${caster_r}**2"/>
          </inertial>
     </visual>
     <collision>
-           <geometry>
-             <sphere radius="${caster_r}"/>
-           </geometry>
+        <origin rpy="${pi/2} 0 0" xyz="0 0 0" />
+        <geometry>
+            <sphere radius="${caster_r}"/>
+        </geometry>
     </collision>
 </link>
@@ -129,11 +138,13 @@
         <inertial>
            <mass value="0.05"/>
+           <origin xyz="0 0 0" />
            <inertia ixx="2/5*${caster_m}*(${caster_r}**2)" ixy="0.0" ixz="0.0" iyy="2/5*${caster_m}*(${caster_r}**2)" iyz="0.0" izz="2/5*${caster_m}*${caster_r}**2"/>
          </inertial>
     </visual>
     <collision>
-           <geometry>
-             <sphere radius="${caster_r}"/>
-           </geometry>
+        <origin rpy="${pi/2} 0 0" xyz="0 0 0" />
+        <geometry>
+            <sphere radius="${caster_r}"/>
+        </geometry>
     </collision>
 </link>

Commit message: Fixed urdf files so that robot spawns correctly within gazebo

File: diff_drive/urdf/ddrive.urdf.xacro (robot description, xacro)
@@ -60,16 +60,18 @@
         </geometry>
         <material name="gray"/>
-        <inertial>
-           <mass value="${wheel_m}"/>
-           <origin rpy="0 0 0" xyz="0 0 0" />
-           <inertia ixx="1/12*${wheel_m}*(3*${wheel_r}**2 + ${wheel_h}**2)" ixy="0.0" ixz="0.0" iyy="1/12*${wheel_m}*(3*${wheel_r}**2 + ${wheel_h}**2)" iyz="0.0" izz="1/2*${wheel_m}*${wheel_r}**2"/>
-         </inertial>
     </visual>
     <collision>
-        <origin rpy="0 0 0" xyz="0 0 0" />
+        <origin rpy="0 ${pi/2} ${pi/2}" xyz="0 0 0" />
         <geometry>
             <cylinder length="${wheel_h}" radius="${wheel_r}"/>
         </geometry>
     </collision>
+    <inertial>
+        <origin rpy="0 0 0" xyz="0 0 0" />
+        <mass value="${wheel_m}"/>
+        <inertia ixx="${1/12*wheel_m*(3*wheel_r**2 + wheel_h**2)}" ixy="0.0" ixz="0.0"
+                 iyy="${1/12*wheel_m*(3*wheel_r**2 + wheel_h**2)}" iyz="0.0"
+                 izz="${1/2*wheel_m*wheel_r**2}"/>
+    </inertial>
 </link>
 <joint name="wheel_left" type="continuous">
@@ -86,16 +88,18 @@
         </geometry>
         <material name="gray"/>
-        <inertial>
-           <mass value="0.2"/>
-           <origin rpy="0 0 0" xyz="0 0 0" />
-           <inertia ixx="1/12*${wheel_m}*(3*${wheel_r}**2 + ${wheel_h}**2)" ixy="0.0" ixz="0.0" iyy="1/12*${wheel_m}*(3*${wheel_r}**2 + ${wheel_h}**2)" iyz="0.0" izz="1/2*${wheel_m}*${wheel_r}**2"/>
-         </inertial>
     </visual>
     <collision>
-        <origin rpy="0 0 0" xyz="0 0 0" />
+        <origin rpy="0 ${pi/2} ${pi/2}" xyz="0 0 0" />
         <geometry>
             <cylinder length="${wheel_h}" radius="${wheel_r}"/>
         </geometry>
     </collision>
+    <inertial>
+        <origin rpy="0 0 0" xyz="0 0 0" />
+        <mass value="${wheel_m}"/>
+        <inertia ixx="${1/12*wheel_m*(3*wheel_r**2 + wheel_h**2)}" ixy="0.0" ixz="0.0"
+                 iyy="${1/12*wheel_m*(3*wheel_r**2 + wheel_h**2)}" iyz="0.0"
+                 izz="${1/2*wheel_m*wheel_r**2}"/>
+    </inertial>
 </link>
 <joint name="caster_top" type="fixed">
@@ -111,9 +115,4 @@
         </geometry>
         <material name="gray"/>
-        <inertial>
-           <mass value="${caster_m}"/>
-           <origin xyz="0 0 0" />
-           <inertia ixx="2/5*${caster_m}*(${caster_r}**2)" ixy="0.0" ixz="0.0" iyy="2/5*${caster_m}*(${caster_r}**2)" iyz="0.0" izz="2/5*${caster_m}*${caster_r}**2"/>
-         </inertial>
     </visual>
     <collision>
@@ -123,4 +122,11 @@
         </geometry>
     </collision>
+    <inertial>
+        <mass value="${caster_m}"/>
+        <origin xyz="0 0 0" />
+        <inertia ixx="${2/5*caster_m*(caster_r**2)}" ixy="0.0" ixz="0.0"
+                 iyy="${2/5*caster_m*(caster_r**2)}" iyz="0.0"
+                 izz="${2/5*caster_m*caster_r**2}"/>
+    </inertial>
 </link>
 <joint name="caster_bottom" type="fixed">
@@ -136,9 +142,4 @@
         </geometry>
         <material name="gray"/>
-        <inertial>
-           <mass value="0.05"/>
-           <origin xyz="0 0 0" />
-           <inertia ixx="2/5*${caster_m}*(${caster_r}**2)" ixy="0.0" ixz="0.0" iyy="2/5*${caster_m}*(${caster_r}**2)" iyz="0.0" izz="2/5*${caster_m}*${caster_r}**2"/>
-         </inertial>
     </visual>
     <collision>
@@ -148,4 +149,11 @@
         </geometry>
     </collision>
+    <inertial>
+        <mass value="${caster_m}"/>
+        <origin xyz="0 0 0" />
+        <inertia ixx="${2/5*caster_m*(caster_r**2)}" ixy="0.0" ixz="0.0"
+                 iyy="${2/5*caster_m*(caster_r**2)}" iyz="0.0"
+                 izz="${2/5*caster_m*caster_r**2}"/>
+    </inertial>
 </link>
 </robot>
