Commit message: Fixed package xml, naming of gazebo xacro, robot spawning but not visible

File: diff_drive/urdf/ddrive.gazebo.xacro (robot description, xacro)
@@ -1,8 +1,8 @@
 <?xml version="1.0"?>
-<robot xmlns:xacro="http://wiki.ros.org/wiki/xacro">
+<robot xmlns:xacro="http://wiki.ros.org/wiki/xacro" name="ddrive">
 <gazebo reference="chassis">
     <material>Gazebo/FlatBlack</material>
 </gazebo>
-<gazebo reference="wheel_right">
+<gazebo reference="right_wheel">
     <material>Gazebo/DarkGrey</material>
     <mu1>999</mu1>
@@ -14,5 +14,5 @@
     <fdir1>1 0 0</fdir1>
 </gazebo>
-<gazebo reference="wheel_left">
+<gazebo reference="left_wheel">
     <material>Gazebo/DarkGrey</material>
     <mu1>999</mu1>
@@ -24,5 +24,5 @@
     <fdir1>1 0 0</fdir1>
 </gazebo>
-<gazebo reference="caster_top">
+<gazebo reference="top_caster">
     <material>Gazebo/Grey</material>
     <mu1>1</mu1>
@@ -34,5 +34,5 @@
     <fdir1>1 0 0</fdir1>
 </gazebo>
-<gazebo reference="caster_bottom">
+<gazebo reference="bottom_caster">
     <material>Gazebo/Grey</material>
     <mu1>1</mu1>

File: diff_drive/urdf/ddrive.urdf.xacro (robot description, xacro)
@@ -1,4 +1,5 @@
 <?xml version="1.0"?>
 <robot xmlns:xacro="http://wiki.ros.org/wiki/xacro" name="ddrive">
+<xacro:include filename="$(find diff_drive)/urdf/ddrive.gazebo.xacro"/>
 <xacro:property name="ddrive" value="$(find diff_drive)/config/ddrive.yaml" />
 <xacro:property name="config" value="${load_yaml(ddrive)}" />
@@ -94,7 +95,7 @@
     <origin xyz="-0.1875 0 0.1" rpy="0 0 0" />
     <parent link="chassis" />
-    <child link="caster_top" />
+    <child link="top_caster" />
 </joint>
-<link name="caster_top">
+<link name="top_caster">
     <visual>
     <origin rpy="${pi/2} 0 0" xyz="0 0 0" />
@@ -117,7 +118,7 @@
     <origin xyz="-0.1875 0 -0.1" rpy="0 0 0" />
     <parent link="chassis" />
-    <child link="caster_bottom" />
+    <child link="bottom_caster" />
 </joint>
-<link name="caster_bottom">
+<link name="bottom_caster">
     <visual>
     <origin rpy="${pi/2} 0 0" xyz="0 0 0" />

Commit message: Configured gazebo plugins and have rviz odom

File: diff_drive/urdf/ddrive.gazebo.xacro (robot description, xacro)
@@ -1,4 +1,13 @@
 <?xml version="1.0"?>
 <robot xmlns:xacro="http://wiki.ros.org/wiki/xacro" name="ddrive">
+<xacro:property name="ddrive" value="$(find diff_drive)/config/ddrive.yaml" />
+<xacro:property name="config" value="${load_yaml(ddrive)}" />
+<xacro:property name="box_l" value="${config['box_l']}" />
+<xacro:property name="box_w" value="${config['box_w']}" />
+<xacro:property name="box_h" value="${config['box_h']}" />
+<xacro:property name="box_m" value="${config['box_m']}" />
+<xacro:property name="wheel_h" value="${config['wheel_h']}" />
+<xacro:property name="wheel_r" value="${config['wheel_r']}" />
+<xacro:property name="wheel_m" value="${config['wheel_m']}" />
 <gazebo reference="chassis">
     <material>Gazebo/FlatBlack</material>
@@ -44,3 +53,25 @@
     <fdir1>1 0 0</fdir1>
 </gazebo>
+<gazebo>
+<plugin name="differential_drive_controller" filename="libgazebo_ros_diff_drive.so">
+<rosDebugLevel>na</rosDebugLevel>
+<alwaysOn>true</alwaysOn>
+<updateRate>100</updateRate>
+<leftJoint>wheel_left</leftJoint>
+<rightJoint>wheel_right</rightJoint>
+<wheelSeparation>${box_w+wheel_h}</wheelSeparation>
+<wheelDiameter>${wheel_r}</wheelDiameter>
+<wheelTorque>20</wheelTorque>
+<commandTopic>diff/cmd_vel</commandTopic>
+<odometryTopic>diff/odom</odometryTopic>
+<odometryFrame>odom</odometryFrame>
+<robotBaseFrame>base_link</robotBaseFrame>
+<publishWheelTF>false</publishWheelTF>
+<publishOdomTF>true</publishOdomTF>
+<publishWheelJointState>true</publishWheelJointState>
+<wheelAcceleration>false</wheelAcceleration>
+<odometrySource>world</odometrySource>
+<publishTf>1</publishTf>
+</plugin>
+</gazebo>
 </robot>
